File: samplehold.kicad_sch (KiCad schematic)
At the start: 95 parts, among them J1 in_1, J10 Synth_power_2x5, J2 out_1, J3 trig_1, J4 in_2, J5 out_2, J6 trig_2, J7 in_3, J8 out_3, J9 trig_3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

Commit message: update to 1.1 with 100nF caps instead of 1nF
Parts:
- C12, C4, C8: value 1n(PP) -> 100n(PP)
Connections:
- net +12V: now also U3.4 (V+); no longer U3.11 (V-)
- net -12V: now also U3.11 (V-); no longer U3.4 (V+)
Other:
- note added: "changed from 1nF to 100nF to improve droop rate"
